File: hardware/mainboard/kicad/power.kicad_sch (KiCad schematic)
At the start: 59 parts, among them J1 XT30PW-M, J2 J_BAT1, J3 J_SW, Q1 AO3401A, Q2 AO3401A, U1 TPS563201DDCR, U2 TPS63070RNMR, U3 AP2112K-3.3TRG1, U6 INA219AIDR

Commit message: Kartonaut: Name, Missionsabzeichen, Bestückungsdruck neu, Lötstopp blau
- Projekt heißt Kartonaut (Karton + Astronaut); Flüge werden hochgezählt, Erstflug = Kartonaut 1
- Abzeichen als Polygone in hardware/mainboard/kicad/logo.py, SVGs in docs/brand/
- spacecode/ -> firmware/, Bodenstation-Repo groundcode -> kartonaut-ground (Links, .gitignore)
- gen_pcb.py silk: Bestückungsdruck nur neu setzen, auf der gerouteten Platine; 1,0 mm Schrift,
  freie Plätze statt Überlappungen, Kurznamen an den Steckern, Testpunkte mit Netznamen,
  kleines Abzeichen vorn; hinten Abzeichen 20 mm und Steckerbelegung
- Stackup JLC04161H-7628 mit blauem Lötstopp im Board, Renders mit Stackup-Farben
- DRC-Druckwarnungen 167 -> 14 (Rest aus Footprint-Umrissen)

Co-Authored-By: Claude Opus 5.5 <noreply@anthropic.com>
Other:
- company: Mission Space -> Kartonaut
Changed lines of the file:
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@@
 		(date "2026-10-21")
 		(rev "B")
-		(company "Mission Space")
+		(company "Kartonaut")
 		(comment 1 "Versorgung: 1S-Pfad (Elektronik) und 2S-Pfad (Aktoren, Pyro)")
 		(comment 2 "erzeugt aus circuit.py (gen_schematic.py)")

Commit message: Mainboard rev B1: Review A1-A8 und Entscheidungen E1-E10 eingearbeitet, 2S-Pfad als F.Cu-Flaechen, 28 Verbindungen offen
Schaltung (circuit.py, ERC 0, Netzliste gegen README §4 OK): Hold-up hinter D1, EN-Teiler 330k/115k,
P-FET-Lastschalter je Akku, Polyfuse je Akku, Kelvin-Shunt mit INA239 an SPI1, BMP390 an SPI1,
74HC138/74HC4051 mit gemeinsamer Adresse, J_STACK 2x10 mit LDO 3V3_EXP, 1S-Lader MCP73831,
J_CHG2, vier Pyro-Kanaele (3/4 DNP), vierter Servo, alle Servos und Rollmotor an VSERVO,
3V3_SENS, eine WS2812B-Kette, Summer Pin 37, E22 NRST Pin 6; 166 Bauteile.

Platine (gen_pcb.py): neue Platzierung, 2S-Pfad, Pyro-Ausgaenge und VSYS_IN als F.Cu-Flaechen mit
Sperrflaechen fuer Freerouting, Strom-Klasse nur F.Cu, IMU-Zone 5 mm, patch mit Umweg ueber In2.
DRC 0 Fehler, Paritaet 0, kein 2S-Netz auf In2; 28 offene Verbindungen, Liste in kicad/README.md §5.5.
Spezifikation README.md und kicad/README.md auf B1 nachgezogen, review_check_layout.py fuer B1.

Co-Authored-By: Claude Opus 5.5 <noreply@anthropic.com>
Parts:
- removed L1: 2.2u Isat>=4A, Inductor_SMD:L_Changjiang_FNR5040S, symbol Device:L
- removed U1: TPS563201DDCR, Package_TO_SOT_SMD:SOT-23-6, symbol Regulator_Switching:TPS563201
- added C23: 10u, Capacitor_SMD:C_0805_2012Metric, symbol Device:C
- added F2: 2A hold, Fuse:Fuse_1812_4532Metric, symbol Device:Polyfuse
- added FB1: 600R@100MHz, Inductor_SMD:L_0603_1608Metric, symbol Device:FerriteBead
- added J17: J_CHG1, Connector_JST:JST_PH_B3B-PH-K_1x03_P2.00mm_Vertical, symbol Connector_Generic:Conn_01x03
- added J18: J_CHG2, Connector_JST:JST_PH_B2B-PH-K_1x02_P2.00mm_Vertical, symbol Connector_Generic:Conn_01x02
- added Q6, Q7: AO3401A, Package_TO_SOT_SMD:SOT-23, symbol Transistor_FET:AO3401A
- added R14: 680k, Resistor_SMD:R_0603_1608Metric, symbol Device:R
- added R15: 130k, Resistor_SMD:R_0603_1608Metric, symbol Device:R
- added R16: 330k, Resistor_SMD:R_0603_1608Metric, symbol Device:R
- added R17: 115k, Resistor_SMD:R_0603_1608Metric, symbol Device:R
- added U11: MCP73831T-2ACI/OT, Package_TO_SOT_SMD:SOT-23-5, symbol Battery_Management:MCP73831-2-OT
- added U14: AP2112K-3.3TRG1, Package_TO_SOT_SMD:SOT-23-5, symbol Regulator_Linear:AP2112K-3.3
- C10: value 22u/10V -> 10u/25V
- C11: value 470u/10V -> 10u/25V; footprint Capacitor_THT:CP_Radial_D8.0mm_P3.50mm -> Capacitor_SMD:C_0805_2012Metric; symbol Device:C_Polarized -> Device:C
- C13, C14: value 10u/25V -> 22u/10V
- C15: value 100n -> 22u/10V; footprint Capacitor_SMD:C_0603_1608Metric -> Capacitor_SMD:C_0805_2012Metric
- C16, C17: value 22u/10V -> 470u/6.3V polymer; footprint Capacitor_SMD:C_0805_2012Metric -> Capacitor_Tantalum_SMD:CP_EIA-7343-31_Kemet-D; symbol Device:C -> Device:C_Polarized
- C18: value 22u/10V -> 1u; footprint Capacitor_SMD:C_0805_2012Metric -> Capacitor_SMD:C_0603_1608Metric
- C19: value 1000u/10V polymer -> 1u; footprint Capacitor_THT:CP_Radial_D8.0mm_P3.50mm -> Capacitor_SMD:C_0603_1608Metric; symbol Device:C_Polarized -> Device:C
- C20: value 1u -> 100u/6.3V; footprint Capacitor_SMD:C_0603_1608Metric -> Capacitor_SMD:C_1210_3225Metric
- C22: value 100u/6.3V -> 1u; footprint Capacitor_SMD:C_1210_3225Metric -> Capacitor_SMD:C_0603_1608Metric
- C3: value 1000u/16V low-ESR -> 100n; footprint Capacitor_THT:CP_Radial_D10.0mm_P5.00mm -> Capacitor_SMD:C_0603_1608Metric; symbol Device:C_Polarized -> Device:C
- C4, C5: value 10u/25V -> 330u/16V polymer; footprint Capacitor_SMD:C_0805_2012Metric -> Capacitor_Tantalum_SMD:CP_EIA-7343-31_Kemet-D; symbol Device:C -> Device:C_Polarized
- C8: value 100n -> 4.7u; footprint Capacitor_SMD:C_0603_1608Metric -> Capacitor_SMD:C_0805_2012Metric
- C9: value 22u/10V -> 4.7u
- F1: value 3A hold -> 3A hold 6A trip; Funktion (none) -> F_BAT2
- NT1: footprint NetTie:NetTie-2_SMD_Pad2.0mm -> NetTie:NetTie-2_SMD_Pad0.5mm
- R10: value 680k -> 1k
- R11: value 130k -> 100k
- R12: value 330k -> 33k
- R13: value 100k -> 2k
- R3: value 33k -> 1k
- R5: value 56k -> 33k
- R6, R7: value 10k -> 10
- R8: value 100k -> 10k
- R9: value 33k -> 100k
- R_SH1: footprint Resistor_SMD:R_2512_6332Metric -> mainboard:R_2512_Kelvin; symbol Device:R -> Device:R_Shunt
- TP5: value 5V_SERVO -> 3V3_RF
- TP6: value 3V3_RF -> 3V3_EXP
- U6: value INA219AIDR -> INA239AIDGSR; footprint Package_SO:SOIC-8_3.9x4.9mm_P1.27mm -> Package_SO:MSOP-10_3x3mm_P0.5mm; symbol Sensor_Energy:INA219AxD -> mainboard:INA239; LCSC C138706 -> (none)
Connections:
- net U1_EN is gone; now on net VBAT2_SENSE: R4.2
- net U1_SW is gone; now on net GND: C8.2
- net 3V3: now also C3.1, U6.6 (VS), FB1.1; no longer C2.1, U6.5 (VS)
- net 3V3_RF: now also C19.1, C20.1, TP5.1; no longer C21.1, C22.1, TP6.1
- net 5V_SYS: now also C13.1, C14.1, C15.1, C21.1, R14.1, U14.1 (VIN), U14.3 (EN); no longer C16.1, C17.1, C19.1, C20.1, R10.1
- net GND: now also C10.2, C11.2, C3.2, C7.2, C9.2, J3.2 (Pin_2), JP1.2 (B), R12.2, R5.2, R8.2, U6.7 (GND), C23.2, J17.2 (Pin_2), R15.2, R17.2, U11.2 (V_{SS}), U14.2 (GND); no longer C2.2, R11.2, R3.2, R7.2, R9.2, U2.6 (FB2), U6.1 (A1), U6.2 (A0), U6.6 (GND)
- net GND_PWR: now also J3.4 (Pin_4), JP2.2 (B), J18.2 (Pin_2); no longer C10.2, C11.2, C3.2, C7.2, C9.2, R6.2
- net Q2_G: now also R8.1; no longer R7.1
- net TEENSY_VIN: now also C16.1, C17.1
- net U2_EN: now also R16.2, R17.1; no longer R12.2, R13.1
- net U2_FB: now also R14.2, R15.1; no longer R10.2, R11.1
- net U2_VAUX: now also C12.1; no longer C15.1
- net VBAT1_SENSE: now also C7.1, R11.2, R12.1; no longer C12.1, R8.2, R9.1
- net VBAT2_RAW: now also J18.1 (Pin_1)
- net VBAT2_REV: now also F1.1; no longer J3.3 (Pin_3), JP2.1 (A)
- net VBAT2_SENSE: now also R5.1; no longer R2.2, R3.1
- net VBAT_PROT: now also Q6.3 (D); no longer J3.4 (Pin_4), JP2.2 (B), R2.1, U6.8 (IN+)
- net VSERVO: now also C5.1, C6.1, R_SH1.4; no longer C3.1, F1.2
- net VSYS_IN: now also C10.1, C11.1, Q7.3 (D), R16.1; no longer C13.1, C14.1, J3.2 (Pin_2), JP1.2 (B), R12.1, R8.1
- removed net 5V_SERVO: C10.1, C11.1, C9.1, R5.1, TP5.1
- net SCL renamed SPI1_MISO
- net SDA: no longer names the net of U6.3 (~{ALERT})
- net U1_BST renamed VBUS_CHG
- net VBUS_CHG: now also J17.1 (Pin_1), U11.4 (V_{DD})
- net U1_FB renamed ISENS_P
- net ISENS_P: now also R_SH1.2; no longer R5.2
- net VBAT1_PROT renamed SW1_G
- net SW1_G: now also R10.2; no longer Q2.2 (S)
- removed net VBAT_MEAS: C5.1, C6.1, C7.1, F1.1, R4.1, R_SH1.2, U6.7 (IN-)
- new net 3V3_EXP: C22.1, TP6.1, U14.5 (VOUT)
- new net 3V3_SENS: C23.1, FB1.2
- new net CHG_PROG: R13.1, U11.5 (PROG)
- new net CHG_STAT: J17.3 (Pin_3), U11.1 (STAT)
- new net CS_INA: U6.1 (~{CS})
- new net INA_INN: C2.2, R7.2, U6.9 (IN-)
- new net INA_INP: C2.1, R6.2, U6.10 (IN+)
- new net ISENS_N: R7.1, R_SH1.3, U6.8 (VBUS)
- new net Q6_G: Q6.1 (G), R2.1, R3.1
- new net Q7_G: Q7.1 (G), R10.1, R9.1
- new net SPI1_MOSI: U6.2 (MOSI)
- new net SPI1_SCK: U6.5 (SCLK)
- new net SW2_G: J3.3 (Pin_3), JP2.1 (A), R3.2
- new net VBAT1_F: C9.1, F2.2, Q7.2 (S), R11.1, R9.2, U11.3 (V_{BAT})
- new net VBAT1_REV: F2.1, Q2.2 (S)
- new net VBAT2_F: F1.2, Q6.2 (S), R2.2, R4.1
- no-connect marks 2 -> 5
Other:
- note added: "1S: Akku, Verpolschutz, Sicherung, Lastschalter"
- note added: "1S: Lader MCP73831"
- note added: "2S: Akku, Verpolschutz, Sicherung, Lastschalter"
- note added: "2S: Spannungsmessung, Shunt und INA239"
- note added: "LDOs 3V3_RF und 3V3_EXP, Sensorinsel, Sternpunkt"
- note added: "Messteiler am Analogmux"
- note added: "Versorgung: 1S-Pfad (Elektronik, Lader) und 2S-Pfad (Aktoren, Pyro), Lastschalter"
- note removed: "1S: Akku, Verpolschutz, Spannungsmessung"
- note removed: "2S: Akku, Verpolschutz, Hauptschalter"
- note removed: "2S: Buck U1 -> 5V_SERVO"
- note removed: "2S: Spannungsmessung und Strommessung INA219"
- note removed: "LDO U3 -> 3V3_RF, Sternpunkt, Testpunkte"
- note removed: "Versorgung: 1S-Pfad (Elektronik) und 2S-Pfad (Aktoren, Pyro)"
- moved on the sheet: C1, C10, C12, C13, C14, C15, C18, C2, C20, C21, C22, C6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
