File: hardware/mainboard/kicad/mainboard.kicad_pcb (KiCad board)
At the start: 4 copper layers, 54 x 120 mm, 166 parts, among them J1 XT30PW-M, J10 J_PYRO2, J11 J_GPS, J12 J_QWIIC, J13 J_CAM, J14 J_LED, J15 J_STACK, J16 J_SERVO4, J17 J_CHG1, J18 J_CHG2, J19 J_PYRO3, J2 J_BAT1, J20 J_PYRO4, J3 J_SW, J4 J_ARM, J5 J_SERVO1, J6 J_SERVO2, J7 J_SERVO3, J8 J_MOT, J9 J_PYRO1, Q1 AO3401A, Q2 AO3401A, Q3 AO3400A, Q4 AO3400A, Q5 AO3400A, Q6 AO3401A, Q7 AO3401A, Q8 AO3400A, Q9 AO3400A, U10 E22-400T22S, U11 MCP73831T-2ACI/OT, U12 74HC138PW, U13 74HC4051PW, U14 AP2112K-3.3TRG1, U15 BMP390, U2 TPS63070RNMR, U3 AP2112K-3.3TRG1, U4 ICM-42688-P, U5 BMP390, U6 INA239AIDGSR, U7 DRV8833PWPR, U8 SN74LV1T34DBVR

Commit message: WIP Handrouting: C6 GND_PWR-Via, 5V_SYS an U14 über B.Cu, PYRO3_NEG (Messleitung über In2), DRC 0/16; Klick-Anleitung
Co-Authored-By: Claude Opus 5.5 <noreply@anthropic.com>
Routing:
- net PYRO3_NEG: track 3.51 -> 8.48 mm
- net 5V_SYS: track 33.9 -> 36.6 mm
- net PYRO3_SENSE: track 76.6 -> 79.1 mm, vias 2 -> 4
- net GND_PWR: track 39.9 -> 41.0 mm, vias 20 -> 21
Changed lines of the file:
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@@
 	)
 	(segment
+		(start 128.4125 65.65)
+		(end 129.17989 65.65)
+		(width 0.3)
+		(layer "F.Cu")
+		(net "GND_PWR")
+	)
+	(segment
 		(start 136.2375 71.25)
 		(end 137.2625 71.25)
@@
 	)
 	(segment
-		(start 128.4125 65.65)
-		(end 129.699999 65.65)
+		(start 129.17989 65.65)
+		(end 129.360483 65.830593)
 		(width 0.3)
 		(layer "F.Cu")
@@
 	)
 	(segment
+		(start 117.58 141.75)
+		(end 118.9 141.75)
+		(width 0.8)
+		(layer "F.Cu")
+		(net "GND_PWR")
+	)
+	(segment
 		(start 148.3625 119.875)
 		(end 149.264061 120.776561)
@@
 	)
 	(via
-		(at 129.699999 65.65)
+		(at 129.360483 65.830593)
 		(size 0.6)
 		(drill 0.3)
@@
 	)
 	(via
+		(at 118.9 141.75)
+		(size 0.8)
+		(drill 0.4)
+		(layers "F.Cu" "B.Cu")
+		(net "GND_PWR")
+	)
+	(via
 		(at 130.2625 71.75)
 		(size 0.6)
@@
 	)
 	(segment
-		(start 135.7232 66.8432)
-		(end 132.4613 66.8432)
+		(start 121.7433 101.7308)
+		(end 122.475 102.4625)
 		(width 0.2)
 		(layer "F.Cu")
@@
 	)
 	(segment
-		(start 121.7433 101.7308)
-		(end 122.475 102.4625)
+		(start 136.5 67.62)
+		(end 135.7232 66.8432)
 		(width 0.2)
 		(layer "F.Cu")
@@
 	)
 	(segment
-		(start 136.5 67.62)
-		(end 135.7232 66.8432)
+		(start 130.4 66.6)
+		(end 130.4 66.7975)
 		(width 0.2)
 		(layer "F.Cu")
@@
 	)
 	(segment
-		(start 132.4613 66.8432)
-		(end 131.4535 67.851)
+		(start 121.4096 103.5279)
+		(end 121.4096 118.3165)
 		(width 0.2)
 		(layer "F.Cu")
@@
 	)
 	(segment
-		(start 121.4096 103.5279)
-		(end 121.4096 118.3165)
+		(start 135.7232 66.8432)
+		(end 134.1432 66.8432)
 		(width 0.2)
 		(layer "F.Cu")
@@
 	)
 	(segment
+		(start 130.4 66.7975)
+		(end 131.4535 67.851)
+		(width 0.2)
+		(layer "F.Cu")
+		(net "PYRO3_SENSE")
+	)
+	(segment
 		(start 122.2 79.948)
 		(end 122.2 98.9625)
@@
 		(net "PYRO3_SENSE")
 	)
+	(segment
+		(start 134.1432 66.8432)
+		(end 133.8 66.5)
+		(width 0.2)
+		(layer "F.Cu")
+		(net "PYRO3_SENSE")
+	)
 	(via
 		(at 128.4048 127.9545)
@@
 	)
 	(via
+		(at 133.8 66.5)
+		(size 0.6)
+		(drill 0.3)
+		(layers "F.Cu" "B.Cu")
+		(net "PYRO3_SENSE")
+	)
+	(via
 		(at 121.6711 118.578)
 		(size 0.6)
@@
 		(net "PYRO3_SENSE")
 	)
+	(via
+		(at 130.4 66.6)
+		(size 0.6)
+		(drill 0.3)
+		(layers "F.Cu" "B.Cu")
+		(net "PYRO3_SENSE")
+	)
 	(segment
 		(start 126.4406 127.9545)
@@
 	)
 	(segment
+		(start 130.5 66.5)
+		(end 130.4 66.6)
+		(width 0.2)
+		(layer "In2.Cu")
+		(net "PYRO3_SENSE")
+	)
+	(segment
 		(start 121.6711 118.578)
 		(end 121.7702 118.6771)
@@
 	)
 	(segment
+		(start 133.8 66.5)
+		(end 130.5 66.5)
+		(width 0.2)
+		(layer "In2.Cu")
+		(net "PYRO3_SENSE")
+	)
+	(segment
 		(start 121.7702 118.6771)
 		(end 121.7702 119.8559)
@@
 	)
 	(segment
+		(start 145 103.1)
+		(end 142.3 103.1)
+		(width 0.5)
+		(layer "B.Cu")
+		(net "5V_SYS")
+	)
+	(segment
 		(start 138.65 80.3)
 		(end 138.65 80.95)
@@
 	)
 	(segment
+		(start 142.3 103.1)
+		(end 142.275 103.075)
+		(width 0.5)
+		(layer "B.Cu")
+		(net "5V_SYS")
+	)
+	(segment
 		(start 145 103.1)
 		(end 145 104.9)
@@
 		(layer "F.Cu")
 		(net "PYRO3_NEG")
+	)
+	(segment
+		(start 133.35 67.7625)
+		(end 133.35 68.4)
+		(width 1)
+		(layer "F.Cu")
+		(net "PYRO3_NEG")
+	)
+	(segment
+		(start 130.2875 64.7)
+		(end 133.35 67.7625)
+		(width 1)
+		(layer "F.Cu")
+		(net "PYRO3_NEG")

Commit message: WIP Handrouting: U7_VINT kürzer neu (28 statt 45 mm, gibt In2 im Mux-Bereich frei), VBAT1_SENSE über B.Cu; DRC 0/15
Co-Authored-By: Claude Opus 5.5 <noreply@anthropic.com>
Routing:
- net U7_VINT: track 50.6 -> 28.2 mm, vias 6 -> 4
- net VBAT1_SENSE: track 26.2 -> 37.2 mm

Commit message: WIP Handrouting: CS_EXT2 neu (5,5 mm B.Cu), VSERVO C35 an die Schiene, VSERVO-Flächen unter J16 vereint; DRC 0/14
Co-Authored-By: Claude Opus 5.5 <noreply@anthropic.com>
Routing:
- net CS_EXT2: track 70.0 -> 67.2 mm, vias 3 -> 5
- net VSERVO: track 16.2 -> 18.2 mm
